Commit message: Add files via upload

File: simpleMod/urdf/simpleMod.urdf (robot description, URDF)
Before this commit: robot simpleMod, 6 links, 5 joints
Links:
- link Component11: geometry collision mesh filename=package://simpleMod/meshes/Component11.stl scale=0.001 0.001 0.001; visual mesh filename=package://simpleMod/meshes/Component11.stl scale=0.001 0.001 0.001
- link Component21: geometry collision mesh filename=package://simpleMod/meshes/Component21.stl scale=0.001 0.001 0.001; visual mesh filename=package://simpleMod/meshes/Component21.stl scale=0.001 0.001 0.001
- link Component31: geometry collision mesh filename=package://simpleMod/meshes/Component31.stl scale=0.001 0.001 0.001; visual mesh filename=package://simpleMod/meshes/Component31.stl scale=0.001 0.001 0.001
- link Component41: geometry collision mesh filename=package://simpleMod/meshes/Component41.stl scale=0.001 0.001 0.001; visual mesh filename=package://simpleMod/meshes/Component41.stl scale=0.001 0.001 0.001
- link Component81: geometry collision mesh filename=package://simpleMod/meshes/Component81.stl scale=0.001 0.001 0.001; visual mesh filename=package://simpleMod/meshes/Component81.stl scale=0.001 0.001 0.001
- link base_link: geometry collision mesh filename=package://simpleMod/meshes/base_link.stl scale=0.001 0.001 0.001; visual mesh filename=package://simpleMod/meshes/base_link.stl scale=0.001 0.001 0.001

Commit message: Add files via upload

File: simpleMod/urdf/simpleMod.urdf (robot description, URDF)
Before this commit: robot simpleMod, 6 links, 5 joints
Links:
- link Component31: geometry collision cylinder length=.09 radius=.15; visual mesh filename=package://simpleMod/meshes/Component31.stl scale=0.001 0.001 0.001
